Commit message: quadruped still kinda fked :(

File: body.urdf (robot description, URDF)
Before this commit: robot robot, 3 links, 2 joints
Links:
- added link BackLowerLeg, mass 1; collision box size=0.2 0.2 1; visual box size=0.2 0.2 1
- added link FrontLowerLeg, mass 1; collision box size=0.2 0.2 1; visual box size=0.2 0.2 1
- added link LeftLeg, mass 1; collision box size=1 0.2 0.2; visual box size=1 0.2 0.2
- added link LeftLowerLeg, mass 1; collision box size=0.2 0.2 1; visual box size=0.2 0.2 1
- added link RightLeg, mass 1; collision box size=1 0.2 0.2; visual box size=1 0.2 0.2
- added link RightLowerLeg, mass 1; collision box size=0.2 0.2 1; visual box size=0.2 0.2 1
- link BackLeg: geometry collision box size=0.2 1 0.2; visual box size=0.2 1 0.2
- link FrontLeg: geometry collision box size=0.2 1 0.2; visual box size=0.2 1 0.2
Joints:
- added joint BackLeg_BackLowerLeg: type revolute, parent BackLeg, child BackLowerLeg, origin xyz=0 -1 0 rpy=0 0 0, axis 1 0 0, limit lower=-3.14159 upper=3.14159 effort=0.0 velocity=0.0
- added joint FrontLeg_FrontLowerLeg: type revolute, parent FrontLeg, child FrontLowerLeg, origin xyz=0 1 0 rpy=0 0 0, axis 1 0 0, limit lower=-3.14159 upper=3.14159 effort=0.0 velocity=0.0
- added joint LeftLeg_LeftLowerLeg: type revolute, parent LeftLeg, child LeftLowerLeg, origin xyz=-1 0 0 rpy=0 0 0, axis 1 0 0, limit lower=-3.14159 upper=3.14159 effort=0.0 velocity=0.0
- added joint RightLeg_RightLowerLeg: type revolute, parent RightLeg, child RightLowerLeg, origin xyz=1 0 0 rpy=0 0 0, axis 1 0 0, limit lower=-3.14159 upper=3.14159 effort=0.0 velocity=0.0
- added joint Torso_LeftLeg: type revolute, parent Torso, child LeftLeg, origin xyz=-0.5 0 1 rpy=0 0 0, axis 1 0 0, limit lower=-3.14159 upper=3.14159 effort=0.0 velocity=0.0
- added joint Torso_RightLeg: type revolute, parent Torso, child RightLeg, origin xyz=0.5 0 1 rpy=0 0 0, axis 1 0 0, limit lower=-3.14159 upper=3.14159 effort=0.0 velocity=0.0
- joint Torso_BackLeg: axis 0 1 0 -> 1 0 0; origin xyz=1 0 1 rpy=0 0 0 -> xyz=0 -0.5 1 rpy=0 0 0
- joint Torso_FrontLeg: axis 0 1 0 -> 1 0 0; origin xyz=2 0 1 rpy=0 0 0 -> xyz=0 0.5 1 rpy=0 0 0

Commit message: turtle created :0

File: body.urdf (robot description, URDF)
Before this commit: robot robot, 9 links, 8 joints
Links:
- removed link BackLeg
- removed link BackLowerLeg
- removed link FrontLeg
- removed link FrontLowerLeg
- removed link LeftLeg
- removed link LeftLowerLeg
- removed link RightLeg
- removed link RightLowerLeg
- added link FootBackLeft, mass 1; collision box size=0.7 0.7 0.25; visual box size=0.7 0.7 0.25
- added link FootBackRight, mass 1; collision box size=0.7 0.7 0.25; visual box size=0.7 0.7 0.25
- added link FootFrontLeft, mass 1; collision box size=0.7 0.7 0.25; visual box size=0.7 0.7 0.25
- added link FootFrontRight, mass 1; collision box size=0.7 0.7 0.25; visual box size=0.7 0.7 0.25
- added link Head, mass 1; collision box size=1 1 1; visual box size=1 1 1
- added link LegBackLeft, mass 1; collision box size=0.625 0.625 0.85; visual box size=0.625 0.625 0.85
- added link LegBackRight, mass 1; collision box size=0.625 0.625 0.85; visual box size=0.625 0.625 0.85
- added link LegFrontLeft, mass 1; collision box size=0.625 0.625 0.85; visual box size=0.625 0.625 0.85
- added link LegFrontRight, mass 1; collision box size=0.625 0.625 0.85; visual box size=0.625 0.625 0.85
- added link Shell1, mass 1; collision box size=2.75 2.25 0.1; visual box size=2.75 2.25 0.1
- added link Shell2, mass 1; collision box size=2.5 2 0.1; visual box size=2.5 2 0.1
- link Torso: geometry collision box size=3 2.5 1.25; visual box size=3 2.5 1.25
Joints:
- removed joint BackLeg_BackLowerLeg
- removed joint FrontLeg_FrontLowerLeg
- removed joint LeftLeg_LeftLowerLeg
- removed joint RightLeg_RightLowerLeg
- removed joint Torso_BackLeg
- removed joint Torso_FrontLeg
- removed joint Torso_LeftLeg
- removed joint Torso_RightLeg
- added joint LegBackLeft_FootBackLeft: type revolute, parent LegBackLeft, child FootBackLeft, origin xyz=0 0 -0.85 rpy=0 0 0, axis 1 1 0, limit lower=-3.14159 upper=3.14159 effort=0.0 velocity=0.0
- added joint LegBackRight_FootBackRight: type revolute, parent LegBackRight, child FootBackRight, origin xyz=0 0 -0.85 rpy=0 0 0, axis 0 1 0, limit lower=-3.14159 upper=3.14159 effort=0.0 velocity=0.0
- added joint LegFrontLeft_FootFrontLeft: type revolute, parent LegFrontLeft, child FootFrontLeft, origin xyz=0 0 -0.85 rpy=0 0 0, axis 0 1 0, limit lower=-3.14159 upper=3.14159 effort=0.0 velocity=0.0
- added joint LegFrontRight_FootFrontRight: type revolute, parent LegFrontRight, child FootFrontRight, origin xyz=0 0 -0.85 rpy=0 0 0, axis 0 1 0, limit lower=-3.14159 upper=3.14159 effort=0.0 velocity=0.0
- added joint Shell1_Shell2: type revolute, parent Shell1, child Shell2, origin xyz=0 0 0.1 rpy=0 0 0, axis 0 1 0, limit lower=-3.14159 upper=3.14159 effort=0.0 velocity=0.0
- added joint Torso_Head: type revolute, parent Torso, child Head, origin xyz=1.25 0 1.675 rpy=0 0 0, axis 0 1 0, limit lower=-3.14159 upper=3.14159 effort=0.0 velocity=0.0
- added joint Torso_LegBackLeft: type revolute, parent Torso, child LegBackLeft, origin xyz=-1.3125 -1.0625 1.1 rpy=0 0 0, axis 1 1 0, limit lower=-3.14159 upper=3.14159 effort=0.0 velocity=0.0
- added joint Torso_LegBackRight: type revolute, parent Torso, child LegBackRight, origin xyz=-1.3125 1.0625 1.1 rpy=0 0 0, axis 1 1 0, limit lower=-3.14159 upper=3.14159 effort=0.0 velocity=0.0
- added joint Torso_LegFrontLeft: type revolute, parent Torso, child LegFrontLeft, origin xyz=1.3125 -1.0625 1.1 rpy=0 0 0, axis 1 1 0, limit lower=-3.14159 upper=3.14159 effort=0.0 velocity=0.0
- added joint Torso_LegFrontRight: type revolute, parent Torso, child LegFrontRight, origin xyz=1.3125 1.0625 1.1 rpy=0 0 0, axis 1 1 0, limit lower=-3.14159 upper=3.14159 effort=0.0 velocity=0.0
- added joint Torso_Shell1: type revolute, parent Torso, child Shell1, origin xyz=0 0 2.1 rpy=0 0 0, axis 0 1 0, limit lower=-3.14159 upper=3.14159 effort=0.0 velocity=0.0

Commit message: turtle evolved :)

File: body.urdf (robot description, URDF)
Before this commit: robot robot, 12 links, 11 joints
Links:
- link FootBackLeft: mass 1 -> 1.0
- link FootBackRight: mass 1 -> 1.0
- link FootFrontLeft: mass 1 -> 1.0
- link FootFrontRight: mass 1 -> 1.0
- link Head: mass 1 -> 1.0
- link LegBackLeft: mass 1 -> 1.0
- link LegBackRight: mass 1 -> 1.0
- link LegFrontLeft: mass 1 -> 1.0
- link LegFrontRight: mass 1 -> 1.0
- link Shell1: mass 1 -> 1.0
- link Shell2: mass 1 -> 1.0
- link Torso: mass 1 -> 40

Commit message: snake yay!

File: body.urdf (robot description, URDF)
Before this commit: robot robot, 12 links, 11 joints
Links:
- removed link FootBackLeft
- removed link FootBackRight
- removed link FootFrontLeft
- removed link FootFrontRight
- removed link Head
- removed link LegBackLeft
- removed link LegBackRight
- removed link LegFrontLeft
- removed link LegFrontRight
- removed link Shell1
- removed link Shell2
- removed link Torso
- added link Link0, mass 1.0; collision box size=0.8038025574165253 0.5996772096235452 0.6273967934103206; visual box size=0.8038025574165253 0.5996772096235452 0.6273967934103206
- added link Link1, mass 1.0; collision box size=0.8489530416311054 0.7390930207170149 0.6910842091677885; visual box size=0.8489530416311054 0.7390930207170149 0.6910842091677885
- added link Link2, mass 1.0; collision box size=0.845821717211829 0.8721462455108546 0.9819258283864102; visual box size=0.845821717211829 0.8721462455108546 0.9819258283864102
- added link Link3, mass 1.0; collision box size=0.847596755882061 0.862582116857011 0.918422939567779; visual box size=0.847596755882061 0.862582116857011 0.918422939567779
Joints:
- removed joint LegBackLeft_FootBackLeft
- removed joint LegBackRight_FootBackRight
- removed joint LegFrontLeft_FootFrontLeft
- removed joint LegFrontRight_FootFrontRight
- removed joint Shell1_Shell2
- removed joint Torso_Head
- removed joint Torso_LegBackLeft
- removed joint Torso_LegBackRight
- removed joint Torso_LegFrontLeft
- removed joint Torso_LegFrontRight
- removed joint Torso_Shell1
- added joint Link0_Link1: type revolute, parent Link0, child Link1, origin xyz=0.8038025574165253 0 0.4909629141932051 rpy=0 0 0, axis 0 1 0, limit lower=-3.14159 upper=3.14159 effort=0.0 velocity=0.0
- added joint Link1_Link2: type revolute, parent Link1, child Link2, origin xyz=0.8489530416311054 0 0.4909629141932051 rpy=0 0 0, axis 0 1 0, limit lower=-3.14159 upper=3.14159 effort=0.0 velocity=0.0
- added joint Link2_Link3: type revolute, parent Link2, child Link3, origin xyz=0.845821717211829 0 0.4909629141932051 rpy=0 0 0, axis 0 1 0, limit lower=-3.14159 upper=3.14159 effort=0.0 velocity=0.0

Commit message: assignment 6 snakey :)

File: body.urdf (robot description, URDF)
Before this commit: robot robot, 4 links, 3 joints
Links:
- added link Link4, mass 1.0; collision box size=0.5122298835093724 0.5799862103170612 0.306505673107648; visual box size=0.5122298835093724 0.5799862103170612 0.306505673107648
- added link Link5, mass 1.0; collision box size=0.4473377904770395 0.7742298445136532 0.7954699817249838; visual box size=0.4473377904770395 0.7742298445136532 0.7954699817249838
- added link Link6, mass 1.0; collision box size=0.47117860254583643 0.4139386526266625 0.7759571507296519; visual box size=0.47117860254583643 0.4139386526266625 0.7759571507296519
- added link Link7, mass 1.0; collision box size=0.9355978404898806 0.8772012977593397 0.5782241542699788; visual box size=0.9355978404898806 0.8772012977593397 0.5782241542699788
- added link Link8, mass 1.0; collision box size=0.4136344231793231 0.6300386019914014 0.3983618924202187; visual box size=0.4136344231793231 0.6300386019914014 0.3983618924202187
- added link Link9, mass 1.0; collision box size=0.7434079021077833 0.7443615638686443 0.8179799428413745; visual box size=0.7434079021077833 0.7443615638686443 0.8179799428413745
- link Link0: geometry collision box size=0.9183356770503452 0.8813695692517824 0.9437101942723225; visual box size=0.9183356770503452 0.8813695692517824 0.9437101942723225
- link Link1: geometry collision box size=0.38356810624266746 0.4909055719835054 0.5426436104012858; visual box size=0.38356810624266746 0.4909055719835054 0.5426436104012858
- link Link2: geometry collision box size=0.5972383493207937 0.482432162449022 0.627725459803201; visual box size=0.5972383493207937 0.482432162449022 0.627725459803201
- link Link3: geometry collision box size=0.6161796404087778 0.3301354002664462 0.8420055680077021; visual box size=0.6161796404087778 0.3301354002664462 0.8420055680077021
Joints:
- added joint Link3_Link4: type revolute, parent Link3, child Link4, origin xyz=0.6161796404087778 0 0 rpy=0 0 0, axis 0 1 0, limit lower=-3.14159 upper=3.14159 effort=0.0 velocity=0.0
- added joint Link4_Link5: type revolute, parent Link4, child Link5, origin xyz=0.5122298835093724 0 0 rpy=0 0 0, axis 0 1 0, limit lower=-3.14159 upper=3.14159 effort=0.0 velocity=0.0
- added joint Link5_Link6: type revolute, parent Link5, child Link6, origin xyz=0.4473377904770395 0 0 rpy=0 0 0, axis 0 1 0, limit lower=-3.14159 upper=3.14159 effort=0.0 velocity=0.0
- added joint Link6_Link7: type revolute, parent Link6, child Link7, origin xyz=0.47117860254583643 0 0 rpy=0 0 0, axis 0 1 0, limit lower=-3.14159 upper=3.14159 effort=0.0 velocity=0.0
- added joint Link7_Link8: type revolute, parent Link7, child Link8, origin xyz=0.9355978404898806 0 0 rpy=0 0 0, axis 0 1 0, limit lower=-3.14159 upper=3.14159 effort=0.0 velocity=0.0
- added joint Link8_Link9: type revolute, parent Link8, child Link9, origin xyz=0.4136344231793231 0 0 rpy=0 0 0, axis 0 1 0, limit lower=-3.14159 upper=3.14159 effort=0.0 velocity=0.0
- joint Link0_Link1: origin xyz=0.8038025574165253 0 0.4909629141932051 rpy=0 0 0 -> xyz=0.4591678385251726 0 0.47185509713616125 rpy=0 0 0
- joint Link1_Link2: origin xyz=0.8489530416311054 0 0.4909629141932051 rpy=0 0 0 -> xyz=0.38356810624266746 0 0 rpy=0 0 0
- joint Link2_Link3: origin xyz=0.845821717211829 0 0.4909629141932051 rpy=0 0 0 -> xyz=0.5972383493207937 0 0 rpy=0 0 0
