Commit message: assignment 7 yay!

File: body.urdf (robot description, URDF)
Before this commit: robot robot, 10 links, 9 joints
Links:
- added link Link10, mass 1.0; collision box size=0.1 0.1 0.1; visual box size=0.1 0.1 0.1
- added link Link11, mass 1.0; collision box size=0.1 0.1 0.1; visual box size=0.1 0.1 0.1
- added link Link12, mass 1.0; collision box size=0.1 0.1 0.1; visual box size=0.1 0.1 0.1
- added link Link13, mass 1.0; collision box size=0.1 0.1 0.1; visual box size=0.1 0.1 0.1
- added link Link14, mass 1.0; collision box size=0.1 0.1 0.1; visual box size=0.1 0.1 0.1
- added link Link15, mass 1.0; collision box size=0.1 0.1 0.1; visual box size=0.1 0.1 0.1
- added link Link16, mass 1.0; collision box size=0.1 0.1 0.1; visual box size=0.1 0.1 0.1
- added link Link17, mass 1.0; collision box size=0.1 0.1 0.1; visual box size=0.1 0.1 0.1
- added link Link18, mass 1.0; collision box size=0.1 0.1 0.1; visual box size=0.1 0.1 0.1
- added link Link19, mass 1.0; collision box size=0.1 0.1 0.1; visual box size=0.1 0.1 0.1
- added link Link20, mass 1.0; collision box size=0.1 0.1 0.1; visual box size=0.1 0.1 0.1
- added link Link21, mass 1.0; collision box size=0.1 0.1 0.1; visual box size=0.1 0.1 0.1
- added link Link22, mass 1.0; collision box size=0.1 0.1 0.1; visual box size=0.1 0.1 0.1
- added link Link23, mass 1.0; collision box size=0.1 0.1 0.1; visual box size=0.1 0.1 0.1
- added link Link24, mass 1.0; collision box size=0.1 0.1 0.1; visual box size=0.1 0.1 0.1
- added link Link25, mass 1.0; collision box size=0.1 0.1 0.1; visual box size=0.1 0.1 0.1
- added link Link26, mass 1.0; collision box size=0.1 0.1 0.1; visual box size=0.1 0.1 0.1
- added link Link27, mass 1.0; collision box size=0.1 0.1 0.1; visual box size=0.1 0.1 0.1
- added link Link28, mass 1.0; collision box size=0.1 0.1 0.1; visual box size=0.1 0.1 0.1
- added link Link29, mass 1.0; collision box size=0.1 0.1 0.1; visual box size=0.1 0.1 0.1
- added link Link30, mass 1.0; collision box size=0.1 0.1 0.1; visual box size=0.1 0.1 0.1
- added link Link31, mass 1.0; collision box size=0.1 0.1 0.1; visual box size=0.1 0.1 0.1
- added link Link32, mass 1.0; collision box size=0.1 0.1 0.1; visual box size=0.1 0.1 0.1
- added link Link33, mass 1.0; collision box size=0.1 0.1 0.1; visual box size=0.1 0.1 0.1
- added link Link34, mass 1.0; collision box size=0.1 0.1 0.1; visual box size=0.1 0.1 0.1
- added link Link35, mass 1.0; collision box size=0.1 0.1 0.1; visual box size=0.1 0.1 0.1
- added link Link36, mass 1.0; collision box size=0.1 0.1 0.1; visual box size=0.1 0.1 0.1
- added link Link37, mass 1.0; collision box size=0.1 0.1 0.1; visual box size=0.1 0.1 0.1
- added link Link38, mass 1.0; collision box size=0.1 0.1 0.1; visual box size=0.1 0.1 0.1
- added link Link39, mass 1.0; collision box size=0.1 0.1 0.1; visual box size=0.1 0.1 0.1
- added link Link40, mass 1.0; collision box size=0.1 0.1 0.1; visual box size=0.1 0.1 0.1
- added link Link41, mass 1.0; collision box size=0.1 0.1 0.1; visual box size=0.1 0.1 0.1
- added link Link42, mass 1.0; collision box size=0.1 0.1 0.1; visual box size=0.1 0.1 0.1
- added link Link43, mass 1.0; collision box size=0.1 0.1 0.1; visual box size=0.1 0.1 0.1
- added link Link44, mass 1.0; collision box size=0.1 0.1 0.1; visual box size=0.1 0.1 0.1
- added link Link45, mass 1.0; collision box size=0.1 0.1 0.1; visual box size=0.1 0.1 0.1
- added link Link46, mass 1.0; collision box size=0.1 0.1 0.1; visual box size=0.1 0.1 0.1
- added link Link47, mass 1.0; collision box size=0.1 0.1 0.1; visual box size=0.1 0.1 0.1
- added link Link48, mass 1.0; collision box size=0.1 0.1 0.1; visual box size=0.1 0.1 0.1
- added link Link49, mass 1.0; collision box size=0.1 0.1 0.1; visual box size=0.1 0.1 0.1
- added link Link50, mass 1.0; collision box size=0.1 0.1 0.1; visual box size=0.1 0.1 0.1
- added link Link51, mass 1.0; collision box size=0.1 0.1 0.1; visual box size=0.1 0.1 0.1
- added link Link52, mass 1.0; collision box size=0.1 0.1 0.1; visual box size=0.1 0.1 0.1
- added link Link53, mass 1.0; collision box size=0.1 0.1 0.1; visual box size=0.1 0.1 0.1
- added link Link54, mass 1.0; collision box size=0.1 0.1 0.1; visual box size=0.1 0.1 0.1
- added link Link55, mass 1.0; collision box size=0.1 0.1 0.1; visual box size=0.1 0.1 0.1
- added link Link56, mass 1.0; collision box size=0.1 0.1 0.1; visual box size=0.1 0.1 0.1
- added link Link57, mass 1.0; collision box size=0.1 0.1 0.1; visual box size=0.1 0.1 0.1
- added link Link58, mass 1.0; collision box size=0.1 0.1 0.1; visual box size=0.1 0.1 0.1
- link Link0: geometry collision box size=0.1 0.1 0.1; visual box size=0.1 0.1 0.1
- link Link1: geometry collision box size=0.1 0.1 0.1; visual box size=0.1 0.1 0.1
- link Link2: geometry collision box size=0.1 0.1 0.1; visual box size=0.1 0.1 0.1
- link Link3: geometry collision box size=0.1 0.1 0.1; visual box size=0.1 0.1 0.1
- link Link4: geometry collision box size=0.1 0.1 0.1; visual box size=0.1 0.1 0.1
- link Link5: geometry collision box size=0.1 0.1 0.1; visual box size=0.1 0.1 0.1
- link Link6: geometry collision box size=0.1 0.1 0.1; visual box size=0.1 0.1 0.1
- link Link7: geometry collision box size=0.1 0.1 0.1; visual box size=0.1 0.1 0.1
- link Link8: geometry collision box size=0.1 0.1 0.1; visual box size=0.1 0.1 0.1
- link Link9: geometry collision box size=0.1 0.1 0.1; visual box size=0.1 0.1 0.1
Joints:
- removed joint Link3_Link4
- removed joint Link4_Link5
- removed joint Link6_Link7
- removed joint Link8_Link9
- added joint Link0_Link16: type revolute, parent Link0, child Link16, origin xyz=0.0 -0.05 1.55 rpy=0 0 0, axis 1 0 0, limit lower=-3.14159 upper=3.14159 effort=0.0 velocity=0.0
- added joint Link0_Link7: type fixed, parent Link0, child Link7, origin xyz=0.05 0.0 1.55 rpy=0 0 0, axis 0 1 0, limit lower=-3.14159 upper=3.14159 effort=0.0 velocity=0.0
- added joint Link10_Link12: type revolute, parent Link10, child Link12, origin xyz=-0.04999999999999999 0.0 -0.050000000000000044 rpy=0 0 0, axis 1 0 0, limit lower=-3.14159 upper=3.14159 effort=0.0 velocity=0.0
- added joint Link10_Link42: type revolute, parent Link10, child Link42, origin xyz=0.0 -0.05 -0.050000000000000044 rpy=0 0 0, axis 0 1 0, limit lower=-3.14159 upper=3.14159 effort=0.0 velocity=0.0
- added joint Link10_Link51: type revolute, parent Link10, child Link51, origin xyz=0.04999999999999999 0.0 -0.050000000000000044 rpy=0 0 0, axis 1 0 0, limit lower=-3.14159 upper=3.14159 effort=0.0 velocity=0.0
- added joint Link11_Link14: type revolute, parent Link11, child Link14, origin xyz=-0.04999999999999999 -0.05 0.0 rpy=0 0 0, axis 1 0 0, limit lower=-3.14159 upper=3.14159 effort=0.0 velocity=0.0
- added joint Link13_Link18: type fixed, parent Link13, child Link18, origin xyz=0.10000000000000002 0.0 0.0 rpy=0 0 0, axis 0 1 0, limit lower=-3.14159 upper=3.14159 effort=0.0 velocity=0.0
- added joint Link14_Link37: type revolute, parent Link14, child Link37, origin xyz=-0.04999999999999999 -0.05 0.0 rpy=0 0 0, axis 0 1 0, limit lower=-3.14159 upper=3.14159 effort=0.0 velocity=0.0
- added joint Link14_Link52: type fixed, parent Link14, child Link52, origin xyz=0.0 -0.10000000000000002 0.0 rpy=0 0 0, axis 0 1 0, limit lower=-3.14159 upper=3.14159 effort=0.0 velocity=0.0
- added joint Link14_Link56: type fixed, parent Link14, child Link56, origin xyz=0.0 -0.05 0.050000000000000044 rpy=0 0 0, axis 0 1 0, limit lower=-3.14159 upper=3.14159 effort=0.0 velocity=0.0
- added joint Link17_Link21: type fixed, parent Link17, child Link21, origin xyz=0.0 -0.05 0.050000000000000044 rpy=0 0 0, axis 0 1 0, limit lower=-3.14159 upper=3.14159 effort=0.0 velocity=0.0
- added joint Link18_Link26: type revolute, parent Link18, child Link26, origin xyz=0.04999999999999999 0.0 -0.050000000000000044 rpy=0 0 0, axis 0 1 0, limit lower=-3.14159 upper=3.14159 effort=0.0 velocity=0.0
- added joint Link18_Link49: type revolute, parent Link18, child Link49, origin xyz=0.04999999999999999 0.0 0.050000000000000044 rpy=0 0 0, axis 1 0 0, limit lower=-3.14159 upper=3.14159 effort=0.0 velocity=0.0
- added joint Link19_Link29: type revolute, parent Link19, child Link29, origin xyz=0.0 0.05000000000000002 -0.050000000000000044 rpy=0 0 0, axis 0 1 0, limit lower=-3.14159 upper=3.14159 effort=0.0 velocity=0.0
- added joint Link19_Link41: type fixed, parent Link19, child Link41, origin xyz=0.05 0.0 -0.050000000000000044 rpy=0 0 0, axis 0 1 0, limit lower=-3.14159 upper=3.14159 effort=0.0 velocity=0.0
- added joint Link1_Link23: type fixed, parent Link1, child Link23, origin xyz=0.0 -0.05 -0.050000000000000044 rpy=0 0 0, axis 0 1 0, limit lower=-3.14159 upper=3.14159 effort=0.0 velocity=0.0
- added joint Link20_Link25: type revolute, parent Link20, child Link25, origin xyz=0.0 0.04999999999999999 -0.050000000000000044 rpy=0 0 0, axis 0 1 0, limit lower=-3.14159 upper=3.14159 effort=0.0 velocity=0.0
- added joint Link20_Link44: type fixed, parent Link20, child Link44, origin xyz=0.05 0.04999999999999999 0.0 rpy=0 0 0, axis 0 1 0, limit lower=-3.14159 upper=3.14159 effort=0.0 velocity=0.0
- added joint Link21_Link54: type revolute, parent Link21, child Link54, origin xyz=-0.05000000000000002 0.0 0.050000000000000044 rpy=0 0 0, axis 0 1 0, limit lower=-3.14159 upper=3.14159 effort=0.0 velocity=0.0
- added joint Link22_Link24: type revolute, parent Link22, child Link24, origin xyz=-0.05000000000000002 0.05 0.0 rpy=0 0 0, axis 0 1 0, limit lower=-3.14159 upper=3.14159 effort=0.0 velocity=0.0
- added joint Link22_Link40: type revolute, parent Link22, child Link40, origin xyz=0.0 0.05 -0.050000000000000044 rpy=0 0 0, axis 1 0 0, limit lower=-3.14159 upper=3.14159 effort=0.0 velocity=0.0
- added joint Link22_Link48: type revolute, parent Link22, child Link48, origin xyz=0.05 0.05 0.0 rpy=0 0 0, axis 1 0 0, limit lower=-3.14159 upper=3.14159 effort=0.0 velocity=0.0
- added joint Link25_Link27: type revolute, parent Link25, child Link27, origin xyz=0.05 0.0 -0.050000000000000044 rpy=0 0 0, axis 1 0 0, limit lower=-3.14159 upper=3.14159 effort=0.0 velocity=0.0
- added joint Link26_Link53: type revolute, parent Link26, child Link53, origin xyz=-0.04999999999999999 0.0 -0.050000000000000044 rpy=0 0 0, axis 1 0 0, limit lower=-3.14159 upper=3.14159 effort=0.0 velocity=0.0
- added joint Link27_Link32: type revolute, parent Link27, child Link32, origin xyz=0.05 0.0 -0.050000000000000044 rpy=0 0 0, axis 1 0 0, limit lower=-3.14159 upper=3.14159 effort=0.0 velocity=0.0
- added joint Link28_Link39: type revolute, parent Link28, child Link39, origin xyz=-0.04999999999999999 0.05 0.0 rpy=0 0 0, axis 0 1 0, limit lower=-3.14159 upper=3.14159 effort=0.0 velocity=0.0
- added joint Link2_Link15: type revolute, parent Link2, child Link15, origin xyz=-0.05 -0.05 0.0 rpy=0 0 0, axis 1 0 0, limit lower=-3.14159 upper=3.14159 effort=0.0 velocity=0.0
- added joint Link2_Link4: type revolute, parent Link2, child Link4, origin xyz=-0.05 0.0 0.050000000000000044 rpy=0 0 0, axis 1 0 0, limit lower=-3.14159 upper=3.14159 effort=0.0 velocity=0.0
- added joint Link2_Link46: type revolute, parent Link2, child Link46, origin xyz=-0.10000000000000002 0.0 0.0 rpy=0 0 0, axis 1 0 0, limit lower=-3.14159 upper=3.14159 effort=0.0 velocity=0.0
- added joint Link2_Link5: type revolute, parent Link2, child Link5, origin xyz=-0.05 0.0 -0.050000000000000044 rpy=0 0 0, axis 1 0 0, limit lower=-3.14159 upper=3.14159 effort=0.0 velocity=0.0
- added joint Link30_Link31: type revolute, parent Link30, child Link31, origin xyz=0.0 -0.05 -0.050000000000000044 rpy=0 0 0, axis 0 1 0, limit lower=-3.14159 upper=3.14159 effort=0.0 velocity=0.0
- added joint Link30_Link45: type revolute, parent Link30, child Link45, origin xyz=0.0 -0.10000000000000002 0.0 rpy=0 0 0, axis 1 0 0, limit lower=-3.14159 upper=3.14159 effort=0.0 velocity=0.0
- added joint Link32_Link55: type revolute, parent Link32, child Link55, origin xyz=0.05000000000000002 0.0 -0.050000000000000044 rpy=0 0 0, axis 0 1 0, limit lower=-3.14159 upper=3.14159 effort=0.0 velocity=0.0
- added joint Link38_Link50: type fixed, parent Link38, child Link50, origin xyz=-0.09999999999999998 0.0 0.0 rpy=0 0 0, axis 0 1 0, limit lower=-3.14159 upper=3.14159 effort=0.0 velocity=0.0
- added joint Link3_Link19: type fixed, parent Link3, child Link19, origin xyz=0.0 0.05 -0.050000000000000044 rpy=0 0 0, axis 0 1 0, limit lower=-3.14159 upper=3.14159 effort=0.0 velocity=0.0
- added joint Link3_Link33: type revolute, parent Link3, child Link33, origin xyz=-0.05000000000000002 0.05 0.0 rpy=0 0 0, axis 0 1 0, limit lower=-3.14159 upper=3.14159 effort=0.0 velocity=0.0
- added joint Link3_Link47: type revolute, parent Link3, child Link47, origin xyz=0.0 0.05 0.050000000000000044 rpy=0 0 0, axis 0 1 0, limit lower=-3.14159 upper=3.14159 effort=0.0 velocity=0.0
- added joint Link3_Link58: type fixed, parent Link3, child Link58, origin xyz=0.0 0.10000000000000002 0.0 rpy=0 0 0, axis 0 1 0, limit lower=-3.14159 upper=3.14159 effort=0.0 velocity=0.0
- added joint Link3_Link9: type fixed, parent Link3, child Link9, origin xyz=0.05 0.05 0.0 rpy=0 0 0, axis 0 1 0, limit lower=-3.14159 upper=3.14159 effort=0.0 velocity=0.0
- added joint Link40_Link43: type fixed, parent Link40, child Link43, origin xyz=0.0 -0.05 -0.050000000000000044 rpy=0 0 0, axis 0 1 0, limit lower=-3.14159 upper=3.14159 effort=0.0 velocity=0.0
- added joint Link4_Link17: type revolute, parent Link4, child Link17, origin xyz=0.0 -0.05 0.050000000000000044 rpy=0 0 0, axis 0 1 0, limit lower=-3.14159 upper=3.14159 effort=0.0 velocity=0.0
- added joint Link4_Link35: type revolute, parent Link4, child Link35, origin xyz=0.0 0.0 0.10000000000000009 rpy=0 0 0, axis 0 1 0, limit lower=-3.14159 upper=3.14159 effort=0.0 velocity=0.0
- added joint Link4_Link38: type revolute, parent Link4, child Link38, origin xyz=-0.05000000000000002 0.0 0.050000000000000044 rpy=0 0 0, axis 1 0 0, limit lower=-3.14159 upper=3.14159 effort=0.0 velocity=0.0
- added joint Link52_Link57: type revolute, parent Link52, child Link57, origin xyz=0.0 -0.04999999999999999 0.050000000000000044 rpy=0 0 0, axis 1 0 0, limit lower=-3.14159 upper=3.14159 effort=0.0 velocity=0.0
- added joint Link5_Link28: type revolute, parent Link5, child Link28, origin xyz=-0.05000000000000002 0.0 -0.050000000000000044 rpy=0 0 0, axis 1 0 0, limit lower=-3.14159 upper=3.14159 effort=0.0 velocity=0.0
- added joint Link6_Link11: type fixed, parent Link6, child Link11, origin xyz=-0.05000000000000002 0.0 -0.050000000000000044 rpy=0 0 0, axis 0 1 0, limit lower=-3.14159 upper=3.14159 effort=0.0 velocity=0.0
- added joint Link6_Link22: type fixed, parent Link6, child Link22, origin xyz=0.0 0.05 -0.050000000000000044 rpy=0 0 0, axis 0 1 0, limit lower=-3.14159 upper=3.14159 effort=0.0 velocity=0.0
- added joint Link7_Link30: type revolute, parent Link7, child Link30, origin xyz=0.05 -0.05 0.0 rpy=0 0 0, axis 0 1 0, limit lower=-3.14159 upper=3.14159 effort=0.0 velocity=0.0
- added joint Link7_Link36: type fixed, parent Link7, child Link36, origin xyz=0.05 0.05 0.0 rpy=0 0 0, axis 0 1 0, limit lower=-3.14159 upper=3.14159 effort=0.0 velocity=0.0
- added joint Link8_Link10: type revolute, parent Link8, child Link10, origin xyz=0.04999999999999999 0.0 -0.050000000000000044 rpy=0 0 0, axis 0 1 0, limit lower=-3.14159 upper=3.14159 effort=0.0 velocity=0.0
- added joint Link9_Link13: type fixed, parent Link9, child Link13, origin xyz=0.1 0.0 0.0 rpy=0 0 0, axis 0 1 0, limit lower=-3.14159 upper=3.14159 effort=0.0 velocity=0.0
- added joint Link9_Link20: type fixed, parent Link9, child Link20, origin xyz=0.05 0.05000000000000002 0.0 rpy=0 0 0, axis 0 1 0, limit lower=-3.14159 upper=3.14159 effort=0.0 velocity=0.0
- added joint Link9_Link34: type revolute, parent Link9, child Link34, origin xyz=0.05 0.0 0.050000000000000044 rpy=0 0 0, axis 0 1 0, limit lower=-3.14159 upper=3.14159 effort=0.0 velocity=0.0
- joint Link0_Link1: axis 0 1 0 -> 1 0 0; origin xyz=0.4591678385251726 0 0.47185509713616125 rpy=0 0 0 -> xyz=0.0 0.0 1.5 rpy=0 0 0
- joint Link1_Link2: axis 0 1 0 -> 1 0 0; origin xyz=0.38356810624266746 0 0 rpy=0 0 0 -> xyz=-0.05 0.0 -0.050000000000000044 rpy=0 0 0
- joint Link2_Link3: origin xyz=0.5972383493207937 0 0 rpy=0 0 0 -> xyz=-0.05 0.05 0.0 rpy=0 0 0
- joint Link5_Link6: origin xyz=0.4473377904770395 0 0 rpy=0 0 0 -> xyz=0.0 0.0 -0.10000000000000009 rpy=0 0 0; type revolute -> fixed
- joint Link7_Link8: origin xyz=0.9355978404898806 0 0 rpy=0 0 0 -> xyz=0.10000000000000002 0.0 0.0 rpy=0 0 0
