Commit message: yuh assignment 7! :)

File: body.urdf (robot description, URDF)
Before this commit: robot robot, 59 links, 58 joints
Links:
- removed link Link19
- removed link Link20
- removed link Link21
- removed link Link22
- removed link Link23
- removed link Link24
- removed link Link25
- removed link Link26
- removed link Link27
- removed link Link28
- removed link Link29
- removed link Link30
- removed link Link31
- removed link Link32
- removed link Link33
- removed link Link34
- removed link Link35
- removed link Link36
- removed link Link37
- removed link Link38
- removed link Link39
- removed link Link40
- removed link Link41
- removed link Link42
- removed link Link43
- removed link Link44
- removed link Link45
- removed link Link46
- removed link Link47
- removed link Link48
- removed link Link49
- removed link Link50
- removed link Link51
- removed link Link52
- removed link Link53
- removed link Link54
- removed link Link55
- removed link Link56
- removed link Link57
- removed link Link58
- link Link0: geometry collision box size=0.8389766661989506 0.453963554633605 0.5849639359655523; visual box size=0.8389766661989506 0.453963554633605 0.5849639359655523
- link Link1: geometry collision box size=0.5466070143580388 0.36668672788930207 0.6498980663623024; visual box size=0.5466070143580388 0.36668672788930207 0.6498980663623024
- link Link10: geometry collision box size=0.532266400533705 0.6029296198736103 0.6065762840122881; visual box size=0.532266400533705 0.6029296198736103 0.6065762840122881
- link Link11: geometry collision box size=0.3680796947121069 0.25942182193394114 0.77908093017489; visual box size=0.3680796947121069 0.25942182193394114 0.77908093017489
- link Link12: geometry collision box size=0.38067939315519744 0.2267581222000284 0.2802308990323772; visual box size=0.38067939315519744 0.2267581222000284 0.2802308990323772
- link Link13: geometry collision box size=0.8397396035435276 0.3662690815039416 0.7874385170836204; visual box size=0.8397396035435276 0.3662690815039416 0.7874385170836204
- link Link14: geometry collision box size=0.4470673322154441 0.5497413019376467 0.2784863225983141; visual box size=0.4470673322154441 0.5497413019376467 0.2784863225983141
- link Link15: geometry collision box size=0.33507549632677747 0.25254340125628477 0.7444250948712121; visual box size=0.33507549632677747 0.25254340125628477 0.7444250948712121
- link Link16: geometry collision box size=0.518901050386691 0.7259055482103389 0.4759191360559103; visual box size=0.518901050386691 0.7259055482103389 0.4759191360559103
- link Link17: geometry collision box size=0.2789531834256986 0.6302854920797372 0.2155710551750848; visual box size=0.2789531834256986 0.6302854920797372 0.2155710551750848
- link Link18: geometry collision box size=0.8702265089900802 0.8737019562371378 0.5592487129376909; visual box size=0.8702265089900802 0.8737019562371378 0.5592487129376909
- link Link2: geometry collision box size=0.9935729025379922 0.6659468624938436 0.9843125510342683; visual box size=0.9935729025379922 0.6659468624938436 0.9843125510342683
- link Link3: geometry collision box size=0.7360598825363007 0.9369171567035506 0.427675742585836; visual box size=0.7360598825363007 0.9369171567035506 0.427675742585836
- link Link4: geometry collision box size=0.9797775393240691 0.7669786156421208 0.5601050050664675; visual box size=0.9797775393240691 0.7669786156421208 0.5601050050664675
- link Link5: geometry collision box size=0.6386485994909773 0.27824613273239385 0.7742795113524856; visual box size=0.6386485994909773 0.27824613273239385 0.7742795113524856
- link Link6: geometry collision box size=0.5017104787624549 0.9663532908415569 0.6646461504802513; visual box size=0.5017104787624549 0.9663532908415569 0.6646461504802513
- link Link7: geometry collision box size=0.6403260977219472 0.8552539575133555 0.4525715172574362; visual box size=0.6403260977219472 0.8552539575133555 0.4525715172574362
- link Link8: geometry collision box size=0.6091581850811478 0.2685666350177671 0.6990115502782892; visual box size=0.6091581850811478 0.2685666350177671 0.6990115502782892
- link Link9: geometry collision box size=0.6527257219194356 0.3847987165516174 0.5588365642747419; visual box size=0.6527257219194356 0.3847987165516174 0.5588365642747419
Joints:
- removed joint Link0_Link16
- removed joint Link0_Link7
- removed joint Link10_Link12
- removed joint Link10_Link42
- removed joint Link10_Link51
- removed joint Link11_Link14
- removed joint Link13_Link18
- removed joint Link14_Link37
- removed joint Link14_Link52
- removed joint Link14_Link56
- removed joint Link17_Link21
- removed joint Link18_Link26
- removed joint Link18_Link49
- removed joint Link19_Link29
- removed joint Link19_Link41
- removed joint Link1_Link2
- removed joint Link1_Link23
- removed joint Link20_Link25
- removed joint Link20_Link44
- removed joint Link21_Link54
- removed joint Link22_Link24
- removed joint Link22_Link40
- removed joint Link22_Link48
- removed joint Link25_Link27
- removed joint Link26_Link53
- removed joint Link27_Link32
- removed joint Link28_Link39
- removed joint Link2_Link15
- removed joint Link2_Link3
- removed joint Link2_Link46
- removed joint Link2_Link5
- removed joint Link30_Link31
- removed joint Link30_Link45
- removed joint Link32_Link55
- removed joint Link38_Link50
- removed joint Link3_Link19
- removed joint Link3_Link33
- removed joint Link3_Link47
- removed joint Link3_Link58
- removed joint Link40_Link43
- removed joint Link4_Link17
- removed joint Link4_Link35
- removed joint Link4_Link38
- removed joint Link52_Link57
- removed joint Link5_Link28
- removed joint Link5_Link6
- removed joint Link6_Link11
- removed joint Link6_Link22
- removed joint Link7_Link30
- removed joint Link7_Link36
- removed joint Link7_Link8
- removed joint Link8_Link10
- removed joint Link9_Link13
- removed joint Link9_Link20
- removed joint Link9_Link34
- added joint Link0_Link13: type revolute, parent Link0, child Link13, origin xyz=0.0 -0.2269817773168025 2.292481967982776 rpy=0 0 0, axis 0 1 0, limit lower=-3.14159 upper=3.14159 effort=0.0 velocity=0.0
- added joint Link0_Link2: type revolute, parent Link0, child Link2, origin xyz=0.0 0.2269817773168025 2.292481967982776 rpy=0 0 0, axis 0 1 0, limit lower=-3.14159 upper=3.14159 effort=0.0 velocity=0.0
- added joint Link0_Link5: type revolute, parent Link0, child Link5, origin xyz=0.0 0.0 2.0 rpy=0 0 0, axis 1 0 0, limit lower=-3.14159 upper=3.14159 effort=0.0 velocity=0.0
- added joint Link13_Link15: type fixed, parent Link13, child Link15, origin xyz=0.0 -0.36626908150394166 0.0 rpy=0 0 0, axis 0 1 0, limit lower=-3.14159 upper=3.14159 effort=0.0 velocity=0.0
- added joint Link14_Link16: type fixed, parent Link14, child Link16, origin xyz=-0.44706733221544415 0.0 0.0 rpy=0 0 0, axis 0 1 0, limit lower=-3.14159 upper=3.14159 effort=0.0 velocity=0.0
- added joint Link1_Link3: type revolute, parent Link1, child Link3, origin xyz=0.5466070143580388 0.0 0.0 rpy=0 0 0, axis 1 0 0, limit lower=-3.14159 upper=3.14159 effort=0.0 velocity=0.0
- added joint Link3_Link10: type fixed, parent Link3, child Link10, origin xyz=0.36802994126815036 0.0 0.2138378712929181 rpy=0 0 0, axis 0 1 0, limit lower=-3.14159 upper=3.14159 effort=0.0 velocity=0.0
- added joint Link3_Link8: type revolute, parent Link3, child Link8, origin xyz=0.36802994126815036 0.4684585783517753 0.0 rpy=0 0 0, axis 0 1 0, limit lower=-3.14159 upper=3.14159 effort=0.0 velocity=0.0
- added joint Link4_Link12: type revolute, parent Link4, child Link12, origin xyz=-0.48988876966203454 -0.3834893078210604 0.0 rpy=0 0 0, axis 0 1 0, limit lower=-3.14159 upper=3.14159 effort=0.0 velocity=0.0
- added joint Link4_Link14: type revolute, parent Link4, child Link14, origin xyz=-0.9797775393240691 0.0 0.0 rpy=0 0 0, axis 1 0 0, limit lower=-3.14159 upper=3.14159 effort=0.0 velocity=0.0
- added joint Link4_Link6: type revolute, parent Link4, child Link6, origin xyz=-0.48988876966203454 0.0 -0.28005250253323366 rpy=0 0 0, axis 0 1 0, limit lower=-3.14159 upper=3.14159 effort=0.0 velocity=0.0
- added joint Link5_Link7: type revolute, parent Link5, child Link7, origin xyz=0.0 -0.13912306636619692 -0.3871397556762428 rpy=0 0 0, axis 1 0 0, limit lower=-3.14159 upper=3.14159 effort=0.0 velocity=0.0
- added joint Link6_Link18: type fixed, parent Link6, child Link18, origin xyz=0.0 0.0 -0.6646461504802514 rpy=0 0 0, axis 0 1 0, limit lower=-3.14159 upper=3.14159 effort=0.0 velocity=0.0
- added joint Link7_Link17: type revolute, parent Link7, child Link17, origin xyz=-0.3201630488609736 -0.4276269787566777 0.0 rpy=0 0 0, axis 0 1 0, limit lower=-3.14159 upper=3.14159 effort=0.0 velocity=0.0
- added joint Link9_Link11: type revolute, parent Link9, child Link11, origin xyz=0.6527257219194356 0.0 0.0 rpy=0 0 0, axis 0 1 0, limit lower=-3.14159 upper=3.14159 effort=0.0 velocity=0.0
- joint Link0_Link1: origin xyz=0.0 0.0 1.5 rpy=0 0 0 -> xyz=0.4194883330994753 0.0 2.292481967982776 rpy=0 0 0
- joint Link2_Link4: origin xyz=-0.05 0.0 0.050000000000000044 rpy=0 0 0 -> xyz=-0.4967864512689961 0.3329734312469218 0.0 rpy=0 0 0
- joint Link3_Link9: axis 0 1 0 -> 1 0 0; origin xyz=0.05 0.05 0.0 rpy=0 0 0 -> xyz=0.7360598825363008 0.0 0.0 rpy=0 0 0; type fixed -> revolute

Commit message: yuh!

File: body.urdf (robot description, URDF)
Before this commit: robot robot, 19 links, 18 joints
Links:
- removed link Link10
- removed link Link11
- removed link Link12
- removed link Link13
- removed link Link14
- removed link Link15
- removed link Link16
- removed link Link17
- removed link Link18
- removed link Link9
- link Link0: geometry collision box size=0.724362858720932 0.4331535957146847 0.13734434053536096; visual box size=0.724362858720932 0.4331535957146847 0.13734434053536096
- link Link1: geometry collision box size=0.6732365997031196 0.5234645983671453 0.6969933508148894; visual box size=0.6732365997031196 0.5234645983671453 0.6969933508148894
- link Link2: geometry collision box size=0.314093182859573 0.21191300217450704 0.43769735161863244; visual box size=0.314093182859573 0.21191300217450704 0.43769735161863244
- link Link3: geometry collision box size=0.5495891810327165 0.9981163968169714 0.21272996992813303; visual box size=0.5495891810327165 0.9981163968169714 0.21272996992813303
- link Link4: geometry collision box size=0.9203666824460559 0.37309323434580655 0.5860383410238836; visual box size=0.9203666824460559 0.37309323434580655 0.5860383410238836
- link Link5: geometry collision box size=0.6034693323122944 0.2944612105070073 0.5359555519501887; visual box size=0.6034693323122944 0.2944612105070073 0.5359555519501887
- link Link6: geometry collision box size=0.8183240516954915 0.8138977309883874 0.19265081554590618; visual box size=0.8183240516954915 0.8138977309883874 0.19265081554590618
- link Link7: geometry collision box size=0.7195710301124663 0.6087007416654023 0.8083710049230411; visual box size=0.7195710301124663 0.6087007416654023 0.8083710049230411
- link Link8: geometry collision box size=0.11017612957618131 0.994683565544593 0.24431219139846905; visual box size=0.11017612957618131 0.994683565544593 0.24431219139846905
Joints:
- removed joint Link0_Link13
- removed joint Link0_Link5
- removed joint Link13_Link15
- removed joint Link14_Link16
- removed joint Link1_Link3
- removed joint Link2_Link4
- removed joint Link3_Link10
- removed joint Link3_Link8
- removed joint Link3_Link9
- removed joint Link4_Link12
- removed joint Link4_Link14
- removed joint Link4_Link6
- removed joint Link5_Link7
- removed joint Link6_Link18
- removed joint Link7_Link17
- removed joint Link9_Link11
- added joint Link0_Link3: type fixed, parent Link0, child Link3, origin xyz=0.0 -0.21657679785734235 1.0686721702676805 rpy=0 0 0, axis 0 1 0, limit lower=-3.14159 upper=3.14159 effort=0.0 velocity=0.0
- added joint Link1_Link5: type revolute, parent Link1, child Link5, origin xyz=-0.6732365997031198 0.0 0.0 rpy=0 0 0, axis 0 1 0, limit lower=-3.14159 upper=3.14159 effort=0.0 velocity=0.0
- added joint Link1_Link7: type revolute, parent Link1, child Link7, origin xyz=-0.33661829985155983 0.26173229918357266 0.0 rpy=0 0 0, axis 0 1 0, limit lower=-3.14159 upper=3.14159 effort=0.0 velocity=0.0
- added joint Link3_Link4: type revolute, parent Link3, child Link4, origin xyz=0.0 -0.4990581984084857 -0.10636498496406654 rpy=0 0 0, axis 1 0 0, limit lower=-3.14159 upper=3.14159 effort=0.0 velocity=0.0
- added joint Link3_Link6: type revolute, parent Link3, child Link6, origin xyz=0.0 -0.9981163968169715 0.0 rpy=0 0 0, axis 0 1 0, limit lower=-3.14159 upper=3.14159 effort=0.0 velocity=0.0
- added joint Link4_Link8: type fixed, parent Link4, child Link8, origin xyz=0.0 0.18654661717290322 -0.2930191705119418 rpy=0 0 0, axis 0 1 0, limit lower=-3.14159 upper=3.14159 effort=0.0 velocity=0.0
- joint Link0_Link1: axis 1 0 0 -> 0 1 0; origin xyz=0.4194883330994753 0.0 2.292481967982776 rpy=0 0 0 -> xyz=-0.362181429360466 0.0 1.0686721702676805 rpy=0 0 0; type revolute -> fixed
- joint Link0_Link2: origin xyz=0.0 0.2269817773168025 2.292481967982776 rpy=0 0 0 -> xyz=0.362181429360466 0.0 1.0686721702676805 rpy=0 0 0; type revolute -> fixed
